Commit message: everything's generated

File: resources/dual_ur5e/spherized.urdf (robot description, URDF)
Before this commit: robot ur5e_robot, 46 links, 45 joints
Links:
- link left_inner_finger_pad: geometry collision sphere radius=0.014593; collision sphere radius=0.014664
- link left_inner_finger_pad_1: geometry collision sphere radius=0.014593; collision sphere radius=0.014664
- link right_inner_finger_pad: geometry collision sphere radius=0.014593; collision sphere radius=0.014664
- link right_inner_finger_pad_1: geometry collision sphere radius=0.014593; collision sphere radius=0.014664
- link robotiq_arg2f_base_link: geometry visual mesh filename=gripper/visual/robotiq_arg2f_85_base_link.dae scale=0.001 0.001 0.001
- link robotiq_arg2f_base_link_1: geometry visual mesh filename=gripper/visual/robotiq_arg2f_85_base_link.dae scale=0.001 0.001 0.001
Joints:
- joint base_fixture_j_base_link: origin xyz=-0.55 0.0 0.0 rpy= 0 0 0 -> xyz=-0.55 0 0.0 rpy=0 0 0
- joint base_fixture_j_base_link_1: origin xyz=0.55 0.0 0.0 rpy= 0 0 0 -> xyz=0.5496187399999999 0.02588207 0.0 rpy= 0 0 -3.105345355171964
- joint base_link-base_link_inertia_1: origin xyz=0 0 0 rpy=0 0 0 -> xyz=0 0 0 rpy=0 0 3.141592653589793
- joint dummy_center_fixed_joint: origin xyz=0 0 0.1725 -> xyz=0 0 0.178
- joint dummy_center_fixed_joint_1: origin xyz=0 0 0.1725 -> xyz=0 0 0.178
- joint finger_joint: axis 1 0 0 -> (none); limit lower=0 upper=0.8 effort=1000 velocity=100.2 -> (none); type revolute -> fixed
- joint finger_joint_1: axis 1 0 0 -> (none); limit lower=0 upper=0.8 effort=1000 velocity=100.2 -> (none); type revolute -> fixed
- joint left_inner_finger_joint: axis 1 0 0 -> (none); limit lower=-0.8 upper=0 effort=1000 velocity=100.2 -> (none); mimic joint=finger_joint multiplier=-1 offset=0 -> (none); type revolute -> fixed
- joint left_inner_finger_joint_1: axis 1 0 0 -> (none); limit lower=-0.8 upper=0 effort=1000 velocity=100.2 -> (none); mimic joint=finger_joint_1 multiplier=-1 offset=0 -> (none); type revolute -> fixed
- joint left_inner_finger_pad_joint: axis 0 0 1 -> (none)
- joint left_inner_finger_pad_joint_1: axis 0 0 1 -> (none)
- joint left_inner_knuckle_joint: axis 1 0 0 -> (none); limit lower=0 upper=0.8 effort=1000 velocity=100.2 -> (none); mimic joint=finger_joint multiplier=1 offset=0 -> (none); type revolute -> fixed
- joint left_inner_knuckle_joint_1: axis 1 0 0 -> (none); limit lower=0 upper=0.8 effort=1000 velocity=100.2 -> (none); mimic joint=finger_joint_1 multiplier=1 offset=0 -> (none); type revolute -> fixed
- joint left_outer_finger_joint: axis 1 0 0 -> (none)
- joint left_outer_finger_joint_1: axis 1 0 0 -> (none)
- joint right_inner_finger_joint: axis 1 0 0 -> (none); limit lower=-0.8 upper=0 effort=1000 velocity=100.2 -> (none); mimic joint=finger_joint multiplier=-1 offset=0 -> (none); type revolute -> fixed
- joint right_inner_finger_joint_1: axis 1 0 0 -> (none); limit lower=-0.8 upper=0 effort=1000 velocity=100.2 -> (none); mimic joint=finger_joint_1 multiplier=-1 offset=0 -> (none); type revolute -> fixed
- joint right_inner_finger_pad_joint: axis 0 0 1 -> (none)
- joint right_inner_finger_pad_joint_1: axis 0 0 1 -> (none)
- joint right_inner_knuckle_joint: axis 1 0 0 -> (none); limit lower=0 upper=0.8 effort=1000 velocity=100.2 -> (none); mimic joint=finger_joint multiplier=1 offset=0 -> (none); type revolute -> fixed
- joint right_inner_knuckle_joint_1: axis 1 0 0 -> (none); limit lower=0 upper=0.8 effort=1000 velocity=100.2 -> (none); mimic joint=finger_joint_1 multiplier=1 offset=0 -> (none); type revolute -> fixed
- joint right_outer_finger_joint: axis 1 0 0 -> (none)
- joint right_outer_finger_joint_1: axis 1 0 0 -> (none)
- joint right_outer_knuckle_joint: axis 1 0 0 -> (none); limit lower=0 upper=0.8 effort=1000 velocity=100.2 -> (none); mimic joint=finger_joint multiplier=1 offset=0 -> (none); type revolute -> fixed
- joint right_outer_knuckle_joint_1: axis 1 0 0 -> (none); limit lower=0 upper=0.8 effort=1000 velocity=100.2 -> (none); mimic joint=finger_joint_1 multiplier=1 offset=0 -> (none); type revolute -> fixed
