Commit message: sphere size increased in GPU allocation

File: resources/dual_ur5e/dual_ur5e_gripper_fixed_fingers.urdf (robot description, URDF)
Before this commit: robot ur5e_robot, 46 links, 45 joints
Links:
- link robotiq_arg2f_base_link: geometry collision mesh filename=gripper/collision/robotiq_arg2f_base_link.stl; visual mesh filename=gripper/visual/robotiq_arg2f_85_base_link.dae scale=0.001 0.001 0.001
- link robotiq_arg2f_base_link_1: geometry collision mesh filename=gripper/collision/robotiq_arg2f_base_link.stl; visual mesh filename=gripper/visual/robotiq_arg2f_85_base_link.dae scale=0.001 0.001 0.001

File: resources/dual_ur5e/spherized.urdf (robot description, URDF)
Before this commit: robot ur5e_robot, 46 links, 45 joints
Links:
- link robotiq_arg2f_base_link: geometry collision sphere radius=0.053503; visual sphere radius=0.053503
- link robotiq_arg2f_base_link_1: geometry collision sphere radius=0.053503; visual sphere radius=0.053503
